File: mcu-bat-power.kicad_sch (KiCad schematic)
At the start: 0 parts

Commit message: First version with all components set and placed
Parts:
- added BT1: BH-18650-B1BA002, Chof747 Footprints:BH18650B1BA002, symbol Chof747 Batteries:BH-18650-B1BA002
- added C1: 1uF, Capacitor_SMD:C_0603_1608Metric_Pad1.08x0.95mm_HandSolder, symbol Device:C
- added C2: 0.1uF, Capacitor_SMD:C_0603_1608Metric_Pad1.08x0.95mm_HandSolder, symbol Device:C
- added C3, C5: 22uF, Capacitor_SMD:C_0603_1608Metric_Pad1.08x0.95mm_HandSolder, symbol Device:C
- added C4: 4u7, Capacitor_SMD:C_0603_1608Metric_Pad1.08x0.95mm_HandSolder, symbol Device:C
- added D1: RED, LED_SMD:LED_0603_1608Metric_Pad1.05x0.95mm_HandSolder, symbol Device:LED
- added D2: GREEN, LED_SMD:LED_0603_1608Metric_Pad1.05x0.95mm_HandSolder, symbol Device:LED
- added D3: SS34A, Chof747 Footprints:DIOM5026X262N, symbol Chof747 passive:SS34A
- added IC1: CN3058E, SOIC127P600X175-9N, symbol Chof747 Battery Management:CN3058E
- added IC2: HY2112, Chof747 Footprints:SOT95P280X145-6N, symbol Chof747 Battery Management:HY2112
- added J1: USB_B_Micro, Chof747 Footprints:Micro USB, symbol Connector:USB_B_Micro
- added J2: INDICATORS, Connector_PinHeader_2.54mm:PinHeader_1x04_P2.54mm_Horizontal, symbol Connector:Conn_01x04_Pin
- added J3: PWR, Connector_PinHeader_2.54mm:PinHeader_1x02_P2.54mm_Horizontal, symbol Connector:Conn_01x02_Pin
- added J4: USB, Connector_PinHeader_2.54mm:PinHeader_1x02_P2.54mm_Horizontal, symbol Connector:Conn_01x02_Pin
- added L1: 22uH, Chof747 Footprints:SMD0740, symbol Device:L
- added Q1: FS8205, FS8205, symbol Chof747 Transistors and Mosfets:FS8205
- added Q2, Q3: 2N7002, Package_TO_SOT_SMD:SOT-23, symbol Transistor_FET:2N7002
- added R1, R12: 1k, Resistor_SMD:R_0603_1608Metric_Pad0.98x0.95mm_HandSolder, symbol Device:R
- added R10: 100, Resistor_SMD:R_0603_1608Metric_Pad0.98x0.95mm_HandSolder, symbol Device:R
- added R11: 7k5, Resistor_SMD:R_0603_1608Metric_Pad0.98x0.95mm_HandSolder, symbol Device:R
- added R13: 2k, Resistor_SMD:R_0603_1608Metric_Pad0.98x0.95mm_HandSolder, symbol Device:R
- added R2: 0, Resistor_SMD:R_0603_1608Metric_Pad0.98x0.95mm_HandSolder, symbol Device:R
- added R3: 2k4 / 1k2, Resistor_SMD:R_0603_1608Metric_Pad0.98x0.95mm_HandSolder, symbol Device:R
- added R4, R7, R8, R9: 10k, Resistor_SMD:R_0603_1608Metric_Pad0.98x0.95mm_HandSolder, symbol Device:R
- added R5, R6: 470k, Resistor_SMD:R_0603_1608Metric_Pad0.98x0.95mm_HandSolder, symbol Device:R
- added SW1: SW_SPDT, Chof747 Footprints:Slide-switch-SS-12D11L7, symbol Switch:SW_SPDT
- added U1: MT3608, Package_TO_SOT_SMD:SOT-23-6, symbol Regulator_Switching:MT3608
Connections:
- new net: J2.3 (Pin_3), Q2.3 (D), R9.2
- new net: R11.2, R12.1, U1.3 (FB)
- new net: J2.2 (Pin_2), Q3.3 (D), R8.2
- new net: C2.1, IC2.6 (VSS), R10.1
- new net: IC2.2 (CS), R13.1
- new net: IC1.2 (ISET), R3.1
- new net: IC2.1 (OD), Q1.6 (G1)
- new net: IC2.3 (OC), Q1.4 (G2)
- new net: IC1.8 (FB), R2.2
- new net: D1.2 (A), D2.2 (A), R1.2
- new net +5V: C5.1, D3.1 (K), J3.1 (Pin_1), R11.1
- new net BAT+: BT1.1 (+), C4.1, IC1.5 (BAT), R10.2, R2.1, SW1.2 (B)
- new net BAT-: BT1.2 (-), C2.2, IC2.5 (VDD), Q1.1 (S1)
- new net BAT_SENSE: J2.4 (Pin_4), R5.1, R6.2
- new net CHG_IND: D1.1 (K), IC1.7 (~{CHRG}), Q3.2 (S), R7.2
- new net GND: C1.2, C3.2, C4.2, C5.2, IC1.1 (TEMP), IC1.3 (GND), IC1.9 (EP), J1.5 (GND), J3.2 (Pin_2), Q1.3 (S2), R12.2, R13.2, R3.2, R6.1, U1.2 (GND)
- new net RDY_IND: D2.1 (K), IC1.6 (~{DONE}), Q2.2 (S), R4.2
- new net USB_N: J1.2 (D-), J4.1 (Pin_1)
- new net USB_P: J1.3 (D+), J4.2 (Pin_2)
- new net VBAT: C3.1, L1.1, R5.2, SW1.1 (A), U1.4 (EN), U1.5 (IN)
- new net VBUS: C1.1, IC1.4 (VIN), J1.1 (VBUS), Q2.1 (G), Q3.1 (G), R1.1, R4.1, R7.1
- new net VREF: J2.1 (Pin_1), R8.1, R9.1
- new net boosted: D3.2 (A), L1.2, U1.1 (SW)
- no-connect marks 0 -> 5
Other:
- note added: "Battery Connector & Switch"
- note added: "Charging"
- note added: "Power & USB Connectors"
- note added: "Sensors"
- note added: "Voltage Boosting"

Commit message: Version 1.0 (sent to fabhouse) + updated readme
Parts:
- added D4: PWR, LED_SMD:LED_0603_1608Metric_Pad1.05x0.95mm_HandSolder, symbol Device:LED
- added D5: USB, LED_SMD:LED_0603_1608Metric_Pad1.05x0.95mm_HandSolder, symbol Device:LED
- added H1, H2, H3, H4: MountingHole, Chof747 Footprints:MountingHole_3.2mm_M3-smallBorder, symbol Mechanical:MountingHole
- added J5: PWR, Chof747_Connectors:pad_1x2_1.5mmx3mm, symbol Connector_Generic:Conn_01x02
- added JP1: A1_H, Jumper:SolderJumper-2_P1.3mm_Open_RoundedPad1.0x1.5mm, symbol Jumper:SolderJumper_2_Open
- added JP2: A1_L, Jumper:SolderJumper-2_P1.3mm_Open_RoundedPad1.0x1.5mm, symbol Jumper:SolderJumper_2_Open
- added JP3: A0_H, Jumper:SolderJumper-2_P1.3mm_Open_RoundedPad1.0x1.5mm, symbol Jumper:SolderJumper_2_Open
- added JP4: A0_L, Jumper:SolderJumper-2_P1.3mm_Open_RoundedPad1.0x1.5mm, symbol Jumper:SolderJumper_2_Open
- added NT1: NetTie_2, NetTie:NetTie-2_SMD_Pad0.5mm, symbol Device:NetTie_2
- added R14: 1k, Resistor_SMD:R_0603_1608Metric_Pad0.98x0.95mm_HandSolder, symbol Device:R
- added TP1: GND, TestPoint:TestPoint_Pad_2.0x2.0mm, symbol Connector:TestPoint
- added TP10: CHG, TestPoint:TestPoint_Pad_2.0x2.0mm, symbol Connector:TestPoint
- added TP2: VBAT, TestPoint:TestPoint_Pad_2.0x2.0mm, symbol Connector:TestPoint
- added TP3: BAT+, TestPoint:TestPoint_Pad_2.0x2.0mm, symbol Connector:TestPoint
- added TP4: BAT-, TestPoint:TestPoint_Pad_2.0x2.0mm, symbol Connector:TestPoint
- added TP5: 5V, TestPoint:TestPoint_Pad_2.0x2.0mm, symbol Connector:TestPoint
- added TP6: FDBK, TestPoint:TestPoint_Pad_2.0x2.0mm, symbol Connector:TestPoint
- added TP7: VBUS, TestPoint:TestPoint_Pad_2.0x2.0mm, symbol Connector:TestPoint
- added TP8: VREF, TestPoint:TestPoint_Pad_2.0x2.0mm, symbol Connector:TestPoint
- added TP9: RDY, TestPoint:TestPoint_Pad_2.0x2.0mm, symbol Connector:TestPoint
- added U2: INA219AxD, Package_SO:SOIC-8_3.9x4.9mm_P1.27mm, symbol Sensor_Energy:INA219AxD
- C3, C5: footprint Capacitor_SMD:C_0603_1608Metric_Pad1.08x0.95mm_HandSolder -> Capacitor_SMD:C_1206_3216Metric_Pad1.33x1.80mm_HandSolder
- J2: footprint Connector_PinHeader_2.54mm:PinHeader_1x04_P2.54mm_Horizontal -> Connector_PinHeader_2.54mm:PinHeader_1x06_P2.54mm_Horizontal; symbol Connector:Conn_01x04_Pin -> Connector:Conn_01x06_Pin
- R5: value 470k -> 0R1; footprint Resistor_SMD:R_0603_1608Metric_Pad0.98x0.95mm_HandSolder -> Resistor_SMD:R_2512_6332Metric_Pad1.40x3.35mm_HandSolder
- R6: value 470k -> 1k
- renumbered BT1 to BAT1
Connections:
- net +5V: now also TP5.1
- net BAT+: now also TP3.1
- net BAT-: now also TP4.1
- net CHG_IND: now also TP10.1
- net GND: now also J2.6 (Pin_6), D4.1 (K), D5.1 (K), J5.2 (Pin_2), JP2.1 (A), JP4.1 (A), NT1.1, TP1.1, U2.6 (GND); no longer R6.1
- net RDY_IND: now also TP9.1
- net VBAT: now also R5.1, R6.1, TP2.1, U2.8 (IN+); no longer C3.1, L1.1, R5.2, U1.4 (EN), U1.5 (IN)
- net VBUS: now also J5.1 (Pin_1), R14.1, TP7.1
- net VREF: now also JP1.2 (B), JP3.2 (B), TP8.1, U2.5 (VS)
- net FDBK: now reaches R11.2, R12.1, U1.3 (FB)
- net FDBK: now also TP6.1
- net at J1.6 (Shield): now also NT1.2
- removed net BAT_SENSE: J2.4 (Pin_4), R5.1, R6.2
- new net: JP3.1 (A), JP4.2 (B), U2.2 (A0)
- new net: D5.2 (A), R14.2
- new net: JP1.1 (A), JP2.2 (B), U2.1 (A1)
- new net: D4.2 (A), R6.2
- new net SCL: J2.5 (Pin_5), U2.4 (SCL)
- new net SDA: J2.4 (Pin_4), U2.3 (SDA)
- new net VBAT_M: C3.1, L1.1, R5.2, U1.4 (EN), U1.5 (IN), U2.7 (IN-)
- no-connect marks 5 -> 4
Other:
- note added: "Battery Protection"
